Commit message: fix: gate LeKiwi motor torque for hardware tests
Keep real-hardware preflight torque-disabled by default, require a separate non-restarting test override to enable torque, and reduce the first-test raw velocity ceiling.

File: ros_depends_ws/src/lekiwi_description/ros2_control/lekiwi_base.ros2_control.xacro (robot description, xacro)
@@ -1,5 +1,5 @@
 <?xml version="1.0"?>
 <robot xmlns:xacro="http://www.ros.org/wiki/xacro">
-  <xacro:macro name="lekiwi_ros2_control" params="hardware_mode">
+  <xacro:macro name="lekiwi_ros2_control" params="hardware_mode enable_motor_torque">
     <ros2_control name="LeKiwiBaseSystem" type="system">
       <hardware>
@@ -13,5 +13,6 @@
           <param name="baud_rate">1000000</param>
           <param name="serial_timeout_ms">20</param>
-          <param name="max_raw_velocity">3000</param>
+          <param name="max_raw_velocity">300</param>
+          <param name="enable_motor_torque">${enable_motor_torque}</param>
           <!-- Joint/controller order is back, right, left. -->
           <param name="back_motor_id">8</param>

File: ros_depends_ws/src/lekiwi_description/urdf/lekiwi_base.urdf.xacro (robot description, xacro)
@@ -2,4 +2,5 @@
 <robot xmlns:xacro="http://www.ros.org/wiki/xacro" name="lekiwi_base">
   <xacro:arg name="hardware_mode" default="mock"/>
+  <xacro:arg name="enable_motor_torque" default="false"/>
   <xacro:property name="base_radius" value="0.125"/>
   <xacro:property name="wheel_radius" value="0.05"/>
@@ -76,4 +77,7 @@
   />
   <xacro:include filename="$(find lekiwi_description)/ros2_control/lekiwi_base.ros2_control.xacro"/>
-  <xacro:lekiwi_ros2_control hardware_mode="$(arg hardware_mode)"/>
+  <xacro:lekiwi_ros2_control
+    hardware_mode="$(arg hardware_mode)"
+    enable_motor_torque="$(arg enable_motor_torque)"
+  />
 </robot>
